File: KiCad/fws/fws.kicad_pcb (KiCad board)
At the start: 2 copper layers, 1 part, among them U1 RP2040

Commit message: Various kicad project updates.
Parts:
- added J1: JST_SM03B-SRSS-TB_LF__SN_, fws:SM03B-SRSS-TB_LF__SN_, F.Cu at (46.0, 47.4)
- added J2: JST_SM03B-SRSS-TB_LF__SN_, fws:SM03B-SRSS-TB_LF__SN_, F.Cu at (71.4, 57.1)
- added U2: RP2040, Package_DFN_QFN:QFN-56-1EP_7x7mm_P0.4mm_EP3.2x3.2mm, F.Cu at (63.0, 60.2)
- added U3: W25Q128JVS, Package_SO:SOIC-8_5.23x5.23mm_P1.27mm, F.Cu at (63.6, 52.1)
- U1: value RP2040 -> MIC5205-3.3YM5; footprint Package_DFN_QFN:QFN-56-1EP_7x7mm_P0.4mm_EP3.2x3.2mm -> Package_TO_SOT_SMD:SOT-23-5
- moved U1 11.4 mm to (71.3, 51.0)
Connections:
- U1 pad 1: Net-(U1-IOVDD-Pad1) -> unconnected-(U1-IN-Pad1)
Other:
- board outline added: 58.4 x 35.6 mm
