File: KiCad/fws/fws.kicad_pcb (KiCad board)
At the start: 2 copper layers, 58.4 x 35.6 mm, 5 parts, among them J1 JST_SM03B-SRSS-TB_LF__SN_, J2 JST_SM03B-SRSS-TB_LF__SN_, U1 MIC5205-3.3YM5, U2 RP2040, U3 W25Q128JVS

Commit message: Added power and usbc.
Parts:
- added D1: 1N5819WS, Diode_SMD:D_SOD-323, F.Cu at (82.8, 45.7)
- J2: value JST_SM03B-SRSS-TB_LF__SN_ -> SM03B-SRSS-TB_LF__SN_
Connections:
- U1 pad 1: unconnected-(U1-IN-Pad1) -> VSYS
- U1 pad 2: unconnected-(U1-GND-Pad2) -> GND
- U1 pad 3: unconnected-(U1-EN-Pad3) -> VSYS
- U1 pad 4: unconnected-(U1-BP-Pad4) -> Net-(U1-BP)
- U1 pad 5: unconnected-(U1-OUT-Pad5) -> +3.3V
- U2 pad 1: Net-(U2-IOVDD-Pad1) -> +3.3V
- U2 pad 10: Net-(U2-IOVDD-Pad1) -> +3.3V
- U2 pad 19: unconnected-(U2-TESTEN-Pad19) -> GND
- U2 pad 22: Net-(U2-IOVDD-Pad1) -> +3.3V
- U2 pad 23: Net-(U2-DVDD-Pad23) -> +1V1
- U2 pad 33: Net-(U2-IOVDD-Pad1) -> +3.3V
- U2 pad 42: Net-(U2-IOVDD-Pad1) -> +3.3V
- U2 pad 43: unconnected-(U2-ADC_AVDD-Pad43) -> +3.3V
- U2 pad 44: unconnected-(U2-VREG_IN-Pad44) -> +3.3V
- U2 pad 45: unconnected-(U2-VREG_VOUT-Pad45) -> +1V1
- U2 pad 46: unconnected-(U2-USB_DM-Pad46) -> Net-(U2-USB_DM)
- U2 pad 47: unconnected-(U2-USB_DP-Pad47) -> Net-(U2-USB_DP)
- U2 pad 48: unconnected-(U2-USB_VDD-Pad48) -> +3.3V
- U2 pad 49: Net-(U2-IOVDD-Pad1) -> +3.3V
- U2 pad 50: Net-(U2-DVDD-Pad23) -> +1V1
- U2 pad 57: unconnected-(U2-GND-Pad57) -> GND

Commit message: Updated pcb.
Parts:
- moved U2 13.2 mm to (52.1, 52.8)
- moved U3 12.7 mm to (54.2, 43.6)
- moved J1 7.67 mm to (40.4, 52.7), turned to -90 degrees
Changed lines of the file:
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@@
   (net 66 "Net-(J2-SHIELD-PadS1)")
   (footprint "Package_DFN_QFN:QFN-56-1EP_7x7mm_P0.4mm_EP3.2x3.2mm" (layer "F.Cu")
-    (at 63.04 60.18)
+    (at 52.1 52.8)
     (descr "QFN, 56 Pin (https://datasheets.raspberrypi.com/rp2040/rp2040-datasheet.pdf#page=634), generated with kicad-footprint-generator ipc_noLead_generator.py")
     (tags "QFN NoLead")
@@
   )
   (footprint "Package_SO:SOIC-8_5.23x5.23mm_P1.27mm" (layer "F.Cu")
-    (at 63.57 52.15)
+    (at 54.2 43.6)
     (descr "SOIC, 8 Pin (http://www.winbond.com/resource-files/w25q32jv%20revg%2003272018%20plus.pdf#page=68), generated with kicad-footprint-generator ipc_gullwing_generator.py")
     (tags "SOIC SO")
@@
   )
   (footprint "fws:SM03B-SRSS-TB_LF__SN_" (layer "F.Cu")
-    (at 45.96 47.445)
-    (property "Reference" "J1" (at -0.635 -1.905 0) (layer "F.SilkS")
-      (effects (font (size 1 1) (thickness 0.15)))
-    )
-    (property "Value" "JST_SM03B-SRSS-TB_LF__SN_" (at 12.065 5.715 0) (layer "F.Fab")
-      (effects (font (size 1 1) (thickness 0.15)))
-    )
-    (property "Footprint" "" (at 0 0 0 unlocked) (layer "F.Fab") hide
-      (effects (font (size 1.27 1.27)))
-    )
-    (property "Datasheet" "" (at 0 0 0 unlocked) (layer "F.Fab") hide
-      (effects (font (size 1.27 1.27)))
-    )
-    (property "Description" "\nConnector Header Surface Mount, Right Angle 3 position 0.039 (1.00mm)\n" (at 45.96 47.445 0) (layer "F.Fab") hide
-      (effects (font (size 1.27 1.27)))
-    )
-    (property "Availability" "In Stock" (at 0 0 0) (layer "F.Fab") hide
-      (effects (font (size 1 1) (thickness 0.15)))
-    )
-    (property "Check_prices" "https://www.snapeda.com/parts/SM03B-SRSS-TB(LF)(SN)/JST+Sales+America+Inc./view-part/?ref=eda" (at 0 0 0) (layer "F.Fab") hide
-      (effects (font (size 1 1) (thickness 0.15)))
-    )
-    (property "MANUFACTURER" "JST" (at 0 0 0) (layer "F.Fab") hide
-      (effects (font (size 1 1) (thickness 0.15)))
-    )
-    (property "MF" "JST Sales" (at 0 0 0) (layer "F.Fab") hide
-      (effects (font (size 1 1) (thickness 0.15)))
-    )
-    (property "MP" "SM03B-SRSS-TB(LF)(SN)" (at 0 0 0) (layer "F.Fab") hide
-      (effects (font (size 1 1) (thickness 0.15)))
-    )
-    (property "Package" "None" (at 0 0 0) (layer "F.Fab") hide
-      (effects (font (size 1 1) (thickness 0.15)))
-    )
-    (property "Price" "None" (at 0 0 0) (layer "F.Fab") hide
-      (effects (font (size 1 1) (thickness 0.15)))
-    )
-    (property "STANDARD" "Manufacturer Recommendation" (at 0 0 0) (layer "F.Fab") hide
-      (effects (font (size 1 1) (thickness 0.15)))
-    )
-    (property "SnapEDA_Link" "https://www.snapeda.com/parts/SM03B-SRSS-TB(LF)(SN)/JST+Sales+America+Inc./view-part/?ref=snap" (at 0 0 0) (layer "F.Fab") hide
+    (at 40.375 52.7 -90)
+    (property "Reference" "J1" (at -0.635 -1.905 90) (layer "F.SilkS")
+      (effects (font (size 1 1) (thickness 0.15)))
+    )
+    (property "Value" "JST_SM03B-SRSS-TB_LF__SN_" (at 12.065 5.715 90) (layer "F.Fab")
+      (effects (font (size 1 1) (thickness 0.15)))
+    )
+    (property "Footprint" "" (at 0 0 -90 unlocked) (layer "F.Fab") hide
+      (effects (font (size 1.27 1.27)))
+    )
+    (property "Datasheet" "" (at 0 0 -90 unlocked) (layer "F.Fab") hide
+      (effects (font (size 1.27 1.27)))
+    )
+    (property "Description" "\nConnector Header Surface Mount, Right Angle 3 position 0.039 (1.00mm)\n" (at 45.96 47.445 90) (layer "F.Fab") hide
+      (effects (font (size 1.27 1.27)))
+    )
+    (property "Availability" "In Stock" (at 0 0 90) (layer "F.Fab") hide
+      (effects (font (size 1 1) (thickness 0.15)))
+    )
+    (property "Check_prices" "https://www.snapeda.com/parts/SM03B-SRSS-TB(LF)(SN)/JST+Sales+America+Inc./view-part/?ref=eda" (at 0 0 90) (layer "F.Fab") hide
+      (effects (font (size 1 1) (thickness 0.15)))
+    )
+    (property "MANUFACTURER" "JST" (at 0 0 90) (layer "F.Fab") hide
+      (effects (font (size 1 1) (thickness 0.15)))
+    )
+    (property "MF" "JST Sales" (at 0 0 90) (layer "F.Fab") hide
+      (effects (font (size 1 1) (thickness 0.15)))
+    )
+    (property "MP" "SM03B-SRSS-TB(LF)(SN)" (at 0 0 90) (layer "F.Fab") hide
+      (effects (font (size 1 1) (thickness 0.15)))
+    )
+    (property "Package" "None" (at 0 0 90) (layer "F.Fab") hide
+      (effects (font (size 1 1) (thickness 0.15)))
+    )
+    (property "Price" "None" (at 0 0 90) (layer "F.Fab") hide
+      (effects (font (size 1 1) (thickness 0.15)))
+    )
+    (property "STANDARD" "Manufacturer Recommendation" (at 0 0 90) (layer "F.Fab") hide
+      (effects (font (size 1 1) (thickness 0.15)))
+    )
+    (property "SnapEDA_Link" "https://www.snapeda.com/parts/SM03B-SRSS-TB(LF)(SN)/JST+Sales+America+Inc./view-part/?ref=snap" (at 0 0 90) (layer "F.Fab") hide
       (effects (font (size 1 1) (thickness 0.15)))
     )
     (attr smd)
+    (fp_line (start -1.3 4.575) (end 1.3 4.575)
+      (stroke (width 0.127) (type solid)) (layer "F.SilkS"))
+    (fp_line (start 2.5 2.6) (end 2.5 0.325)
+      (stroke (width 0.127) (type solid)) (layer "F.SilkS"))
     (fp_line (start -2.5 0.325) (end -2.5 2.6)
       (stroke (width 0.127) (type solid)) (layer "F.SilkS"))
     (fp_line (start -1.615 0.325) (end -2.5 0.325)
       (stroke (width 0.127) (type solid)) (layer "F.SilkS"))
-    (fp_line (start -1.3 4.575) (end 1.3 4.575)
-      (stroke (width 0.127) (type solid)) (layer "F.SilkS"))
     (fp_line (start 2.5 0.325) (end 1.615 0.325)
-      (stroke (width 0.127) (type solid)) (layer "F.SilkS"))
-    (fp_line (start 2.5 2.6) (end 2.5 0.325)
       (stroke (width 0.127) (type solid)) (layer "F.SilkS"))
     (fp_circle (center -1.8 -0.4) (end -1.7 -0.4)
       (stroke (width 0.3) (type solid)) (fill none) (layer "F.SilkS"))
+    (fp_line (start -3.15 5.025) (end -3.15 -1.025)
+      (stroke (width 0.05) (type solid)) (layer "F.CrtYd"))
+    (fp_line (start 3.15 5.025) (end -3.15 5.025)
+      (stroke (width 0.05) (type solid)) (layer "F.CrtYd"))
     (fp_line (start -3.15 -1.025) (end 3.15 -1.025)
       (stroke (width 0.05) (type solid)) (layer "F.CrtYd"))
-    (fp_line (start -3.15 5.025) (end -3.15 -1.025)
-      (stroke (width 0.05) (type solid)) (layer "F.CrtYd"))
     (fp_line (start 3.15 -1.025) (end 3.15 5.025)
       (stroke (width 0.05) (type solid)) (layer "F.CrtYd"))
-    (fp_line (start 3.15 5.025) (end -3.15 5.025)
-      (stroke (width 0.05) (type solid)) (layer "F.CrtYd"))
+    (fp_line (start -2.5 4.575) (end -2.5 0.325)
+      (stroke (width 0.127) (type solid)) (layer "F.Fab"))
+    (fp_line (start 2.5 4.575) (end -2.5 4.575)
+      (stroke (width 0.127) (type solid)) (layer "F.Fab"))
     (fp_line (start -2.5 0.325) (end 2.5 0.325)
       (stroke (width 0.127) (type solid)) (layer "F.Fab"))
-    (fp_line (start -2.5 4.575) (end -2.5 0.325)
-      (stroke (width 0.127) (type solid)) (layer "F.Fab"))
     (fp_line (start 2.5 0.325) (end 2.5 4.575)
-      (stroke (width 0.127) (type solid)) (layer "F.Fab"))
-    (fp_line (start 2.5 4.575) (end -2.5 4.575)
       (stroke (width 0.127) (type solid)) (layer "F.Fab"))
     (fp_circle (center -1.8 -0.4) (end -1.7 -0.4)
       (stroke (width 0.3) (type solid)) (fill none) (layer "F.Fab"))
-    (pad "1" smd rect (at -1 0 90) (size 1.55 0.6) (layers "F.Cu" "F.Paste" "F.Mask")
+    (pad "1" smd rect (at -1 0) (size 1.55 0.6) (layers "F.Cu" "F.Paste" "F.Mask")
       (net 59 "unconnected-(J1-Pad1)") (pinfunction "1") (pintype "passive") (solder_mask_margin 0.102)
     )
-    (pad "2" smd rect (at 0 0 90) (size 1.55 0.6) (layers "F.Cu" "F.Paste" "F.Mask")
+    (pad "2" smd rect (at 0 0) (size 1.55 0.6) (layers "F.Cu" "F.Paste" "F.Mask")
       (net 60 "unconnected-(J1-Pad2)") (pinfunction "2") (pintype "passive") (solder_mask_margin 0.102)
     )
-    (pad "3" smd rect (at 1 0 90) (size 1.55 0.6) (layers "F.Cu" "F.Paste" "F.Mask")
+    (pad "3" smd rect (at 1 0) (size 1.55 0.6) (layers "F.Cu" "F.Paste" "F.Mask")
       (net 61 "unconnected-(J1-Pad3)") (pinfunction "3") (pintype "passive") (solder_mask_margin 0.102)
     )
-    (pad "S1" smd rect (at -2.3 3.875 180) (size 1.2 1.8) (layers "F.Cu" "F.Paste" "F.Mask")
+    (pad "S1" smd rect (at -2.3 3.875 90) (size 1.2 1.8) (layers "F.Cu" "F.Paste" "F.Mask")
       (net 62 "Net-(J1-SHIELD-PadS1)") (pinfunction "SHIELD") (pintype "passive") (solder_mask_margin 0.102)
     )
-    (pad "S2" smd rect (at 2.3 3.875 180) (size 1.2 1.8) (layers "F.Cu" "F.Paste" "F.Mask")
+    (pad "S2" smd rect (at 2.3 3.875 90) (size 1.2 1.8) (layers "F.Cu" "F.Paste" "F.Mask")
       (net 62 "Net-(J1-SHIELD-PadS1)") (pinfunction "SHIELD") (pintype "passive") (solder_mask_margin 0.102)
     )

Commit message: Updated pcb.
Parts:
- moved D1 46.6 mm to (41.0, 66.5)
- moved U1 30.6 mm to (42.0, 60.0)
- moved J2 16.2 mm to (67.9, 41.3)
Changed lines of the file:
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@@
   )
   (footprint "Package_TO_SOT_SMD:SOT-23-5" (layer "F.Cu")
-    (at 71.32 50.99)
+    (at 42.0375 59.95)
     (descr "SOT, 5 Pin (https://www.jedec.org/sites/default/files/docs/Mo-178c.PDF variant AA), generated with kicad-footprint-generator ipc_gullwing_generator.py")
     (tags "SOT TO_SOT_SMD")
@@
   )
   (footprint "Diode_SMD:D_SOD-323" (layer "F.Cu")
-    (at 82.77 45.72)
+    (at 41.05 66.5)
     (descr "SOD-323")
     (tags "SOD-323")
@@
   )
   (footprint "fws:SM03B-SRSS-TB_LF__SN_" (layer "F.Cu")
-    (at 71.36 57.085)
+    (at 67.9 41.3)
     (property "Reference" "J2" (at -0.635 -1.905 0) (layer "F.SilkS")
       (effects (font (size 1 1) (thickness 0.15)))

Commit message: Updated pcb.
Parts:
- moved J2 18.8 mm to (61.8, 59.1)
- moved U2 5.41 mm to (51.9, 58.2)
Changed lines of the file:
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@@
   (net 66 "Net-(J2-SHIELD-PadS1)")
   (footprint "Package_DFN_QFN:QFN-56-1EP_7x7mm_P0.4mm_EP3.2x3.2mm" (layer "F.Cu")
-    (at 52.1 52.8)
+    (at 51.8625 58.2)
     (descr "QFN, 56 Pin (https://datasheets.raspberrypi.com/rp2040/rp2040-datasheet.pdf#page=634), generated with kicad-footprint-generator ipc_noLead_generator.py")
     (tags "QFN NoLead")
@@
   )
   (footprint "fws:SM03B-SRSS-TB_LF__SN_" (layer "F.Cu")
-    (at 67.9 41.3)
+    (at 61.8 59.1)
     (property "Reference" "J2" (at -0.635 -1.905 0) (layer "F.SilkS")
       (effects (font (size 1 1) (thickness 0.15)))

Commit message: Updated pcb.
Parts:
- moved U2 19.4 mm to (68.1, 47.5)
- moved J2 17.1 mm to (44.7, 58.2)
- moved J1 10.2 mm to (40.4, 42.5)
- moved U1 8.61 mm to (46.8, 67.2)
Changed lines of the file:
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@@
   (net 66 "Net-(J2-SHIELD-PadS1)")
   (footprint "Package_DFN_QFN:QFN-56-1EP_7x7mm_P0.4mm_EP3.2x3.2mm" (layer "F.Cu")
-    (at 51.8625 58.2)
+    (at 68.0625 47.5)
     (descr "QFN, 56 Pin (https://datasheets.raspberrypi.com/rp2040/rp2040-datasheet.pdf#page=634), generated with kicad-footprint-generator ipc_noLead_generator.py")
     (tags "QFN NoLead")
@@
   )
   (footprint "Package_TO_SOT_SMD:SOT-23-5" (layer "F.Cu")
-    (at 42.0375 59.95)
+    (at 46.7625 67.15)
     (descr "SOT, 5 Pin (https://www.jedec.org/sites/default/files/docs/Mo-178c.PDF variant AA), generated with kicad-footprint-generator ipc_gullwing_generator.py")
     (tags "SOT TO_SOT_SMD")
@@
   )
   (footprint "fws:SM03B-SRSS-TB_LF__SN_" (layer "F.Cu")
-    (at 61.8 59.1)
+    (at 44.7 58.2)
     (property "Reference" "J2" (at -0.635 -1.905 0) (layer "F.SilkS")
       (effects (font (size 1 1) (thickness 0.15)))
@@
   )
   (footprint "fws:SM03B-SRSS-TB_LF__SN_" (layer "F.Cu")
-    (at 40.375 52.7 -90)
+    (at 40.375 42.5 -90)
     (property "Reference" "J1" (at -0.635 -1.905 90) (layer "F.SilkS")
       (effects (font (size 1 1) (thickness 0.15)))

Commit message: Updated pcb.
Parts:
- added C1: 100nF, Capacitor_SMD:C_0603_1608Metric_Pad1.08x0.95mm_HandSolder, F.Cu at (78.8, 44.7)
- added C10: 100nF, Capacitor_SMD:C_0603_1608Metric_Pad1.08x0.95mm_HandSolder, F.Cu at (83.1, 49.7)
- added C11: 4.7uF, Capacitor_SMD:C_0603_1608Metric_Pad1.08x0.95mm_HandSolder, F.Cu at (83.1, 52.2)
- added C12: 100nF, Capacitor_SMD:C_0603_1608Metric_Pad1.08x0.95mm_HandSolder, F.Cu at (83.1, 54.8)
- added C13: 100nF, Capacitor_SMD:C_0603_1608Metric_Pad1.08x0.95mm_HandSolder, F.Cu at (83.1, 57.3)
- added C14: 100nF, Capacitor_SMD:C_0603_1608Metric_Pad1.08x0.95mm_HandSolder, F.Cu at (83.1, 59.8)
- added C15: 100nF, Capacitor_SMD:C_0603_1608Metric_Pad1.08x0.95mm_HandSolder, F.Cu at (87.5, 44.7)
- added C16: 100nF, Capacitor_SMD:C_0603_1608Metric_Pad1.08x0.95mm_HandSolder, F.Cu at (87.5, 47.2)
- added C17: 100nF, Capacitor_SMD:C_0603_1608Metric_Pad1.08x0.95mm_HandSolder, F.Cu at (87.5, 49.7)
- added C18: 100nF, Capacitor_SMD:C_0603_1608Metric_Pad1.08x0.95mm_HandSolder, F.Cu at (87.5, 52.2)
- added C2: 4.7uF, Capacitor_SMD:C_0603_1608Metric_Pad1.08x0.95mm_HandSolder, F.Cu at (78.8, 47.2)
- added C3: 10uF, Capacitor_SMD:C_0603_1608Metric_Pad1.08x0.95mm_HandSolder, F.Cu at (78.8, 49.7)
- added C4: 27pF, Capacitor_SMD:C_0603_1608Metric_Pad1.08x0.95mm_HandSolder, F.Cu at (78.8, 52.2)
- added C5: 27pF, Capacitor_SMD:C_0603_1608Metric_Pad1.08x0.95mm_HandSolder, F.Cu at (78.8, 54.8)
- added C6: 470pF, Capacitor_SMD:C_0603_1608Metric_Pad1.08x0.95mm_HandSolder, F.Cu at (78.8, 57.3)
- added C7: 10uF, Capacitor_SMD:C_0603_1608Metric_Pad1.08x0.95mm_HandSolder, F.Cu at (78.8, 59.8)
- added C8: 4.7uF, Capacitor_SMD:C_0603_1608Metric_Pad1.08x0.95mm_HandSolder, F.Cu at (83.1, 44.7)
- added C9: 100nF, Capacitor_SMD:C_0603_1608Metric_Pad1.08x0.95mm_HandSolder, F.Cu at (83.1, 47.2)
- added R1: 1K, Capacitor_SMD:C_0603_1608Metric_Pad1.08x0.95mm_HandSolder, F.Cu at (87.5, 54.8)
- added R2: 10K, Capacitor_SMD:C_0603_1608Metric_Pad1.08x0.95mm_HandSolder, F.Cu at (87.5, 57.3)
- added R3: R, Capacitor_SMD:C_0603_1608Metric_Pad1.08x0.95mm_HandSolder, F.Cu at (87.5, 59.8)
- added R4: R, Capacitor_SMD:C_0603_1608Metric_Pad1.08x0.95mm_HandSolder, F.Cu at (91.8, 44.7)
- added R5: 10K, Capacitor_SMD:C_0603_1608Metric_Pad1.08x0.95mm_HandSolder, F.Cu at (91.8, 47.2)
- added R6: 27R, Capacitor_SMD:C_0603_1608Metric_Pad1.08x0.95mm_HandSolder, F.Cu at (91.8, 49.7)
- added R7: 27R, Capacitor_SMD:C_0603_1608Metric_Pad1.08x0.95mm_HandSolder, F.Cu at (91.8, 52.2)
- added S1: ~, FWS:s13131-1536, F.Cu at (81.8, 62.9)
- U1: value MIC5205-3.3YM5 -> W25Q128JVS; footprint Package_TO_SOT_SMD:SOT-23-5 -> Package_SO:SOIC-8_5.23x5.23mm_P1.27mm
- U2: value RP2040 -> MIC5205-3.3YM5; footprint Package_DFN_QFN:QFN-56-1EP_7x7mm_P0.4mm_EP3.2x3.2mm -> Package_TO_SOT_SMD:SOT-23-5
- U3: value W25Q128JVS -> RP2040; footprint Package_SO:SOIC-8_5.23x5.23mm_P1.27mm -> Package_DFN_QFN:QFN-56-1EP_7x7mm_P0.4mm_EP3.2x3.2mm
Connections:
- J2 pad 1: unconnected-(J2-Pad1) -> /SWCLK
- J2 pad 2: unconnected-(J2-Pad2) -> GND
- J2 pad 3: unconnected-(J2-Pad3) -> /SWD
- J2 pad S1: Net-(J2-SHIELD-PadS1) -> GND
- J2 pad S2: Net-(J2-SHIELD-PadS1) -> GND
- U1 pad 1: VSYS -> /QSPI_SS
- U1 pad 2: GND -> /QSPI_SD1
- U1 pad 3: VSYS -> /QSPI_SD2
- U1 pad 4: Net-(U1-BP) -> GND
- U1 pad 5: +3.3V -> /QSPI_SD0
- U2 pad 1: +3.3V -> VSYS
- U2 pad 2: unconnected-(U2-GPIO0-Pad2) -> GND
- U2 pad 3: unconnected-(U2-GPIO1-Pad3) -> VSYS
- U2 pad 4: unconnected-(U2-GPIO2-Pad4) -> Net-(U2-BP)
- U2 pad 5: unconnected-(U2-GPIO3-Pad5) -> +3.3V
- U3 pad 1: unconnected-(U3-~{CS}-Pad1) -> +3.3V

Commit message: Updated PCB
Parts:
- added C19: 22uF, Capacitor_SMD:C_0603_1608Metric_Pad1.08x0.95mm_HandSolder, F.Cu at (34.5, 20.9)
- added C20: 100nF, Capacitor_SMD:C_0603_1608Metric_Pad1.08x0.95mm_HandSolder, F.Cu at (34.5, 23.4)
- added C21: 100nF, Capacitor_SMD:C_0603_1608Metric_Pad1.08x0.95mm_HandSolder, F.Cu at (34.5, 25.9)
- C12: value 100nF -> 4.7uF
- C17: value 100nF -> 100n
- C6: value 470pF -> 4.7uF
- C7: value 10uF -> 470pF
- C8: value 4.7uF -> 100nF
- C9: value 100nF -> 10uF
Connections:
- C11 pad 1: +3.3V -> Net-(S1-Vcp)
- C6 pad 1: Net-(U2-BP) -> +1V1
- C7 pad 1: +3.3V -> Net-(U2-BP)
- C9 pad 1: +1V1 -> +3.3V
- S1 pad 1: unconnected-(S1-CLK-Pad1) -> /CLK
- S1 pad 2: unconnected-(S1-Vcp-Pad2) -> Net-(S1-Vcp)
- S1 pad 3: unconnected-(S1-GND-Pad3) -> GND
- S1 pad 4: unconnected-(S1-Video-Pad4) -> /VIDEO
- S1 pad 5: unconnected-(S1-EOS-Pad5) -> /EOS
- S1 pad 6: unconnected-(S1-Vdd-Pad6) -> +3.3V
- S1 pad 7: unconnected-(S1-Trig-Pad7) -> /TRIG
- S1 pad 8: unconnected-(S1-ST-Pad8) -> /ST
- U3 pad 34: unconnected-(U3-GPIO22-Pad34) -> /EOS
- U3 pad 35: unconnected-(U3-GPIO23-Pad35) -> /TRIG
- U3 pad 36: unconnected-(U3-GPIO24-Pad36) -> /ST
- U3 pad 37: unconnected-(U3-GPIO25-Pad37) -> /CLK
- U3 pad 38: unconnected-(U3-GPIO26_ADC0-Pad38) -> /VIDEO
