File: KiCad/fws/fws.kicad_sch (KiCad schematic)
At the start: 35 parts, among them J1 USB_C_Receptacle_USB2.0, J2 SM03B-SRSS-TB_LF__SN_, U1 W25Q128JVS, U2 MIC5205-3.3YM5, U3 RP2040, Y1 12MHz

Commit message: Updated schematics.
Connections:
- net VIDEO: now reaches U3.38 (GPIO26_ADC0)
- net VIDEO: now also S1.4 (Video)
Changed lines of the file:
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@@
   (no_connect (at 45.72 55.88))
   (no_connect (at 45.72 53.34))
+  (wire (pts (xy 161.29 34.29) (xy 167.64 34.29))
+    (stroke (width 0) (type default))
+  )
   (wire (pts (xy 171.45 71.12) (xy 179.07 71.12))
     (stroke (width 0) (type default))
@@
   )
   (wire (pts (xy 124.46 151.13) (xy 132.08 151.13))
+    (stroke (width 0) (type default))
+  )
+  (wire (pts (xy 182.88 153.67) (xy 189.23 153.67))
     (stroke (width 0) (type default))
   )
@@
     (effects (font (size 1.27 1.27)) (justify left bottom))
   )
+  (label "VIDEO" (at 161.29 34.29 0) (fields_autoplaced)
+    (effects (font (size 1.27 1.27)) (justify left bottom))
+  )
   (label "QSPI_SD2" (at 31.75 119.38 0) (fields_autoplaced)
     (effects (font (size 1.27 1.27)) (justify left bottom))
@@
     (effects (font (size 1.27 1.27)) (justify left bottom))
   )
+  (label "VIDEO" (at 189.23 153.67 180) (fields_autoplaced)
+    (effects (font (size 1.27 1.27)) (justify right bottom))
+  )
   (label "QSPI_SD1" (at 120.65 110.49 0) (fields_autoplaced)

Commit message: Updated schematics.
Connections:
- net EOS: now reaches U3.34 (GPIO22)
- net EOS: now also S1.5 (EOS)
- net TRIG: now reaches U3.35 (GPIO23)
- net TRIG: now also S1.7 (Trig)
- net ST: now reaches U3.36 (GPIO24)
- net ST: now also S1.8 (ST)
- net CLK: now reaches U3.37 (GPIO25)
- net CLK: now also S1.1 (CLK)
Changed lines of the file:
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@@
+    (stroke (width 0) (type default))
+  )
+  (wire (pts (xy 161.29 26.67) (xy 167.64 26.67))
     (stroke (width 0) (type default))
   )
@@
     (stroke (width 0) (type default))
   )
+  (wire (pts (xy 182.88 148.59) (xy 189.23 148.59))
+    (stroke (width 0) (type default))
+  )
   (wire (pts (xy 120.65 107.95) (xy 132.08 107.95))
     (stroke (width 0) (type default))
@@
     (stroke (width 0) (type default))
   )
+  (wire (pts (xy 185.42 34.29) (xy 191.77 34.29))
+    (stroke (width 0) (type default))
+  )
   (wire (pts (xy 201.93 68.58) (xy 201.93 71.12))
     (stroke (width 0) (type default))
@@
     (stroke (width 0) (type default))
   )
+  (wire (pts (xy 182.88 146.05) (xy 189.23 146.05))
+    (stroke (width 0) (type default))
+  )
   (wire (pts (xy 154.94 77.47) (xy 154.94 57.15))
     (stroke (width 0) (type default))
@@
     (stroke (width 0) (type default))
   )
+  (wire (pts (xy 182.88 143.51) (xy 189.23 143.51))
+    (stroke (width 0) (type default))
+  )
   (wire (pts (xy 38.1 167.64) (xy 38.1 170.18))
     (stroke (width 0) (type default))
@@
     (stroke (width 0) (type default))
   )
+  (wire (pts (xy 182.88 140.97) (xy 189.23 140.97))
+    (stroke (width 0) (type default))
+  )
   (wire (pts (xy 45.72 25.4) (xy 50.8 25.4))
     (stroke (width 0) (type default))
@@
     (stroke (width 0) (type default))
   )
+  (wire (pts (xy 185.42 26.67) (xy 191.77 26.67))
+    (stroke (width 0) (type default))
+  )
   (wire (pts (xy 76.2 25.4) (xy 76.2 34.29))
     (stroke (width 0) (type default))
@@
   )
   (wire (pts (xy 144.78 68.58) (xy 144.78 71.12))
+    (stroke (width 0) (type default))
+  )
+  (wire (pts (xy 185.42 29.21) (xy 191.77 29.21))
     (stroke (width 0) (type default))
   )
@@
     (effects (font (size 1.27 1.27)) (justify left bottom))
   )
+  (label "TRIG" (at 189.23 143.51 180) (fields_autoplaced)
+    (effects (font (size 1.27 1.27)) (justify right bottom))
+  )
+  (label "TRIG" (at 191.77 29.21 180) (fields_autoplaced)
+    (effects (font (size 1.27 1.27)) (justify right bottom))
+  )
   (label "VIDEO" (at 161.29 34.29 0) (fields_autoplaced)
     (effects (font (size 1.27 1.27)) (justify left bottom))
@@
     (effects (font (size 1.27 1.27)) (justify left bottom))
   )
+  (label "EOS" (at 191.77 34.29 180) (fields_autoplaced)
+    (effects (font (size 1.27 1.27)) (justify right bottom))
+  )
   (label "QSPI_SCLK" (at 120.65 118.11 0) (fields_autoplaced)
     (effects (font (size 1.27 1.27)) (justify left bottom))
@@
     (effects (font (size 1.27 1.27)) (justify left bottom))
   )
+  (label "CLK" (at 161.29 26.67 0) (fields_autoplaced)
+    (effects (font (size 1.27 1.27)) (justify left bottom))
+  )
   (label "QSPI_SD3" (at 31.75 121.92 0) (fields_autoplaced)
     (effects (font (size 1.27 1.27)) (justify left bottom))
   )
+  (label "ST" (at 189.23 146.05 180) (fields_autoplaced)
+    (effects (font (size 1.27 1.27)) (justify right bottom))
+  )
+  (label "EOS" (at 189.23 140.97 180) (fields_autoplaced)
+    (effects (font (size 1.27 1.27)) (justify right bottom))
+  )
   (label "QSPI_SD3" (at 120.65 115.57 0) (fields_autoplaced)
     (effects (font (size 1.27 1.27)) (justify left bottom))
@@
     (effects (font (size 1.27 1.27)) (justify left bottom))
   )
+  (label "ST" (at 191.77 26.67 180) (fields_autoplaced)
+    (effects (font (size 1.27 1.27)) (justify right bottom))
+  )
   (label "QSPI_SS" (at 31.75 109.22 0) (fields_autoplaced)
     (effects (font (size 1.27 1.27)) (justify left bottom))
@@
     (effects (font (size 1.27 1.27)) (justify left bottom))
   )
+  (label "CLK" (at 189.23 148.59 180) (fields_autoplaced)
+    (effects (font (size 1.27 1.27)) (justify right bottom))
+  )
   (label "QSPI_SD0" (at 120.65 107.95 0) (fields_autoplaced)

Commit message: Updated schematics.
Parts:
- added C?: 4.7uF, Capacitor_SMD:C_0603_1608Metric_Pad1.08x0.95mm_HandSolder, symbol FWS:C
- added C?: 22uF, Capacitor_SMD:C_0603_1608Metric_Pad1.08x0.95mm_HandSolder, symbol FWS:C_Polarized
- added C?: 100n, Capacitor_SMD:C_0603_1608Metric_Pad1.08x0.95mm_HandSolder, symbol FWS:C
Connections:
- net +3.3V: now also S1.6 (Vdd), C?.1, C?.1; no longer S1.2 (Vcp)
- net GND: now also C?.2, C?.2, C?.2
- new net: C?.1, S1.2 (Vcp)
Other:
- moved on the sheet: S1
