File: KiCad/s13131_breakout/s13131_breakout.kicad_pcb (KiCad board)
At the start: 2 copper layers, 24.7 x 20.4 mm, 3 parts, among them J1 Conn_01x07_Pin

Commit message: Updated breakout.
Parts:
- added C2: 100n, Capacitor_SMD:C_0805_2012Metric, B.Cu at (45.1, 54.8)
- added C3: 22u 25v, Capacitor_SMD:CP_Elec_5x5.4, F.Cu at (61.6, 52.1)
- moved J1 8.25 mm to (66.8, 50.9)
Routing:
- net +3.3V: track 16.2 -> 27.2 mm
- net /CLK: track 23.7 -> 33.3 mm
- net /Video: track 15.6 -> 23.9 mm
- net /ST: track 20.4 -> 28.7 mm
- net /EOS: track 13.1 -> 21.4 mm
- net /Trig: track 18.8 -> 27.1 mm
Other:
- board size 24.7 x 20.4 mm -> 33 x 20.4 mm

Commit message: Updated breakout pcb.
Routing:
- net /EOS: track 21.4 -> 19.8 mm
Changed lines of the file:
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@@
   (gr_line (start 36 48.5) (end 56 68.5)
     (stroke (width 0.1) (type default)) (layer "F.Fab"))
-  (segment (start 65.155 57.6) (end 66.75 56.005) (width 0.25) (layer "F.Cu") (net 1))
+  (segment (start 64.495 56.005) (end 66.75 56.005) (width 0.25) (layer "F.Cu") (net 1))
+  (segment (start 55.8 57.6) (end 62.9 57.6) (width 0.25) (layer "F.Cu") (net 1))
+  (segment (start 42.4 58.6) (end 41.35 58.6) (width 0.25) (layer "F.Cu") (net 1))
   (segment (start 52.15 53.95) (end 55.8 57.6) (width 0.25) (layer "F.Cu") (net 1))
+  (segment (start 62.9 57.6) (end 64.495 56.005) (width 0.25) (layer "F.Cu") (net 1))
+  (segment (start 41.35 53.95) (end 52.15 53.95) (width 0.25) (layer "F.Cu") (net 1))
   (segment (start 41.35 58.6) (end 41.35 53.95) (width 0.25) (layer "F.Cu") (net 1))
-  (segment (start 42.4 58.6) (end 41.35 58.6) (width 0.25) (layer "F.Cu") (net 1))
-  (segment (start 55.8 57.6) (end 65.155 57.6) (width 0.25) (layer "F.Cu") (net 1))
-  (segment (start 41.35 53.95) (end 52.15 53.95) (width 0.25) (layer "F.Cu") (net 1))
   (segment (start 66.705 66.12) (end 66.75 66.165) (width 0.25) (layer "F.Cu") (net 2))
   (segment (start 49.6 58.6) (end 49.6 64.8) (width 0.25) (layer "F.Cu") (net 2))
   (segment (start 49.6 64.8) (end 50.92 66.12) (width 0.25) (layer "F.Cu") (net 2))
   (segment (start 50.92 66.12) (end 66.705 66.12) (width 0.25) (layer "F.Cu") (net 2))
+  (segment (start 65.775 63.625) (end 66.75 63.625) (width 0.25) (layer "F.Cu") (net 3))
   (segment (start 49.6 57.16) (end 52.16 57.16) (width 0.25) (layer "F.Cu") (net 3))
-  (segment (start 55.55 63.15) (end 56.025 63.625) (width 0.25) (layer "F.Cu") (net 3))
-  (segment (start 55.55 60.55) (end 55.55 63.15) (width 0.25) (layer "F.Cu") (net 3))
-  (segment (start 56.025 63.625) (end 66.75 63.625) (width 0.25) (layer "F.Cu") (net 3))
   (segment (start 52.16 57.16) (end 55.55 60.55) (width 0.25) (layer "F.Cu") (net 3))
+  (segment (start 62.7 60.55) (end 65.775 63.625) (width 0.25) (layer "F.Cu") (net 3))
+  (segment (start 55.55 60.55) (end 62.7 60.55) (width 0.25) (layer "F.Cu") (net 3))
   (segment (start 51.6 54.5) (end 55.645 58.545) (width 0.25) (layer "F.Cu") (net 4))
   (segment (start 42.4 57.16) (end 42.4 54.5) (width 0.25) (layer "F.Cu") (net 4))
   (segment (start 55.645 58.545) (end 66.75 58.545) (width 0.25) (layer "F.Cu") (net 4))
   (segment (start 42.4 54.5) (end 51.6 54.5) (width 0.25) (layer "F.Cu") (net 4))
-  (segment (start 57.085 61.085) (end 51.05 55.05) (width 0.25) (layer "F.Cu") (net 5))
-  (segment (start 66.75 61.085) (end 57.085 61.085) (width 0.25) (layer "F.Cu") (net 5))
   (segment (start 44.3 55.05) (end 44.3 57.16) (width 0.25) (layer "F.Cu") (net 5))
+  (segment (start 55.4 59.4) (end 51.05 55.05) (width 0.25) (layer "F.Cu") (net 5))
   (segment (start 51.05 55.05) (end 44.3 55.05) (width 0.25) (layer "F.Cu") (net 5))
+  (segment (start 64.485 61.085) (end 62.8 59.4) (width 0.25) (layer "F.Cu") (net 5))
+  (segment (start 66.75 61.085) (end 64.485 61.085) (width 0.25) (layer "F.Cu") (net 5))
+  (segment (start 62.8 59.4) (end 55.4 59.4) (width 0.25) (layer "F.Cu") (net 5))
   (segment (start 44.3 58.6) (end 44.3 60.1) (width 0.25) (layer "F.Cu") (net 6))
   (via (at 44.3 60.1) (size 0.8) (drill 0.4) (layers "F.Cu" "B.Cu") (net 6))
