File: KiCad/s13131_breakout/s13131_breakout.kicad_sch (KiCad schematic)
At the start: 1 part

Commit message: Updated breakout.
Parts:
- added C1: 1uF, Capacitor_SMD:C_0805_2012Metric, symbol FWS:C
- added J1: Conn_01x07_Pin, Connector_PinHeader_2.54mm:PinHeader_1x07_P2.54mm_Vertical, symbol FWS:Conn_01x07_Pin
- renumbered S13131 to S1
Connections:
- net CLK: now reaches S1.1 (CLK)
- net CLK: now also J1.3 (Pin_3)
- net at S1.2 (Vcp): now also C1.1
- net GND: now reaches S1.3 (GND)
- net GND: now also C1.2, J1.2 (Pin_2)
- net Video: now reaches S1.4 (Video)
- net Video: now also J1.7 (Pin_7)
- net EOS: now reaches S1.5 (EOS)
- net EOS: now also J1.6 (Pin_6)
- net +3.3V: now reaches S1.6 (Vdd)
- net +3.3V: now also J1.1 (Pin_1)
- net Trig: now reaches S1.7 (Trig)
- net Trig: now also J1.5 (Pin_5)
- net ST: now reaches S1.8 (ST)
- net ST: now also J1.4 (Pin_4)
Other:
- moved on the sheet: S1

Commit message: Updated breakout schematics.
Parts:
- added C?: 100n, Capacitor_SMD:C_0805_2012Metric, symbol FWS:C
- added C?: 22u 25v, symbol FWS:C_Polarized
Connections:
- net +3.3V: now also C?.1, C?.1
- net GND: now also C?.2, C?.2
Changed lines of the file:
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@@
 (kicad_sch (version 20230819) (generator eeschema)
   (paper "A4")
+  (junction (at 100.33 62.23) (diameter 0) (color 0 0 0 0)
+  )
   (wire (pts (xy 90.17 57.15) (xy 95.25 57.15))
     (stroke (width 0) (type default))
@@
     (stroke (width 0) (type default))
   )
+  (wire (pts (xy 107.95 63.5) (xy 107.95 62.23))
+    (stroke (width 0) (type default))
+  )
   (wire (pts (xy 59.69 71.12) (xy 59.69 72.39))
     (stroke (width 0) (type default))
   )
+  (wire (pts (xy 107.95 62.23) (xy 100.33 62.23))
+    (stroke (width 0) (type default))
+  )
   (wire (pts (xy 33.02 68.58) (xy 38.1 68.58))
     (stroke (width 0) (type default))
   )
+  (wire (pts (xy 107.95 71.12) (xy 107.95 72.39))
+    (stroke (width 0) (type default))
+  )
   (wire (pts (xy 33.02 66.04) (xy 38.1 66.04))
     (stroke (width 0) (type default))
@@
   )
   (wire (pts (xy 90.17 64.77) (xy 95.25 64.77))
+    (stroke (width 0) (type default))
+  )
+  (wire (pts (xy 100.33 62.23) (xy 100.33 63.5))
+    (stroke (width 0) (type default))
+  )
+  (wire (pts (xy 100.33 71.12) (xy 100.33 72.39))
     (stroke (width 0) (type default))
   )
@@
     )
   )
+  (symbol (lib_id "FWS:C") (at 100.33 67.31 0) (unit 1)
+    (exclude_from_sim no) (in_bom yes) (on_board yes) (dnp no)
+    (property "Reference" "C?" (at 100.965 64.77 0)
+      (effects (font (size 1.27 1.27)) (justify left))
+    )
+    (property "Value" "100n" (at 100.965 69.85 0)
+      (effects (font (size 1.27 1.27)) (justify left))
+    )
+    (property "Footprint" "Capacitor_SMD:C_0805_2012Metric" (at 101.2952 71.12 0)
+      (effects (font (size 1.27 1.27)) hide)
+    )
+    (property "Datasheet" "~" (at 100.33 67.31 0)
+      (effects (font (size 1.27 1.27)) hide)
+    )
+    (property "Description" "Unpolarized capacitor" (at 100.33 67.31 0)
+      (effects (font (size 1.27 1.27)) hide)
+    )
+    (pin "1")
+    (pin "2")
+    (instances
+      (project "s13131_breakout"
+        (path "/9b830ee6-51b1-4891-8c58-db3625e8ab27"
+          (reference "C?") (unit 1)
+        )
+      )
+    )
+  )
   (symbol (lib_id "FWS:GND") (at 44.45 60.96 0) (unit 1)
     (exclude_from_sim no) (in_bom yes) (on_board yes) (dnp no)
@@
         (path "/9b830ee6-51b1-4891-8c58-db3625e8ab27"
           (reference "#PWR02") (unit 1)
+        )
+      )
+    )
+  )
+  (symbol (lib_id "FWS:C_Polarized") (at 107.95 67.31 0) (unit 1)
+    (exclude_from_sim no) (in_bom yes) (on_board yes) (dnp no)
+    (property "Reference" "C?" (at 108.585 64.77 0)
+      (effects (font (size 1.27 1.27)) (justify left))
+    )
+    (property "Value" "22u 25v" (at 108.585 69.85 0)
+      (effects (font (size 1.27 1.27)) (justify left))
+    )
+    (property "Footprint" "" (at 108.9152 71.12 0)
+      (effects (font (size 1.27 1.27)) hide)
+    )
+    (property "Datasheet" "~" (at 107.95 67.31 0)
+      (effects (font (size 1.27 1.27)) hide)
+    )
+    (property "Description" "Polarized capacitor" (at 107.95 67.31 0)
+      (effects (font (size 1.27 1.27)) hide)
+    )
+    (pin "1")
+    (pin "2")
+    (instances
+      (project "s13131_breakout"
+        (path "/9b830ee6-51b1-4891-8c58-db3625e8ab27"
+          (reference "C?") (unit 1)
         )
       )
@@
     )
   )
+  (symbol (lib_id "FWS:GND") (at 100.33 72.39 0) (unit 1)
+    (exclude_from_sim no) (in_bom yes) (on_board yes) (dnp no)
+    (property "Reference" "#PWR06" (at 100.33 78.74 0)
+      (effects (font (size 1.27 1.27)) hide)
+    )
+    (property "Value" "GND" (at 100.33 76.2 0)
+      (effects (font (size 1.27 1.27)))
+    )
+    (property "Footprint" "" (at 100.33 72.39 0)
+      (effects (font (size 1.27 1.27)) hide)
+    )
+    (property "Datasheet" "" (at 100.33 72.39 0)
+      (effects (font (size 1.27 1.27)) hide)
+    )
+    (property "Description" "Power symbol creates a global label with name \"GND\" , ground" (at 100.33 72.39 0)
+      (effects (font (size 1.27 1.27)) hide)
+    )
+    (pin "1")
+    (instances
+      (project "s13131_breakout"
+        (path "/9b830ee6-51b1-4891-8c58-db3625e8ab27"
+          (reference "#PWR06") (unit 1)
+        )
+      )
+    )
+  )
   (symbol (lib_id "FWS:+3.3V") (at 44.45 58.42 0) (unit 1)
     (exclude_from_sim no) (in_bom yes) (on_board yes) (dnp no)
@@
         )
       )
+    )
+  )
+  (symbol (lib_id "FWS:GND") (at 107.95 72.39 0) (unit 1)
+    (exclude_from_sim no) (in_bom yes) (on_board yes) (dnp no)
+    (property "Reference" "#PWR07" (at 107.95 78.74 0)
+      (effects (font (size 1.27 1.27)) hide)
+    )
+    (property "Value" "GND" (at 107.95 76.2 0)
+      (effects (font (size 1.27 1.27)))
+    )
+    (property "Footprint" "" (at 107.95 72.39 0)
+      (effects (font (size 1.27 1.27)) hide)
+    )
+    (property "Datasheet" "" (at 107.95 72.39 0)
+      (effects (font (size 1.27 1.27)) hide)
+    )
+    (property "Description" "Power symbol creates a global label with name \"GND\" , ground" (at 107.95 72.39 0)
+      (effects (font (size 1.27 1.27)) hide)
+    )
+    (pin "1")
+    (instances
+      (project "s13131_breakout"
+        (path "/9b830ee6-51b1-4891-8c58-db3625e8ab27"
+          (reference "#PWR07") (unit 1)
+        )
+      )

Commit message: Updated breakout.
Parts:
- C3: renamed from C?; footprint (none) -> Capacitor_SMD:CP_Elec_5x5.4
- gave numbers to parts that had none: 1
Changed lines of the file:
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@@
   (symbol (lib_id "FWS:C") (at 100.33 67.31 0) (unit 1)
     (exclude_from_sim no) (in_bom yes) (on_board yes) (dnp no)
-    (property "Reference" "C?" (at 100.965 64.77 0)
+    (property "Reference" "C2" (at 100.965 64.77 0)
       (effects (font (size 1.27 1.27)) (justify left))
     )
@@
       (project "s13131_breakout"
         (path "/9b830ee6-51b1-4891-8c58-db3625e8ab27"
-          (reference "C?") (unit 1)
+          (reference "C2") (unit 1)
         )
       )
@@
   (symbol (lib_id "FWS:C_Polarized") (at 107.95 67.31 0) (unit 1)
     (exclude_from_sim no) (in_bom yes) (on_board yes) (dnp no)
-    (property "Reference" "C?" (at 108.585 64.77 0)
+    (property "Reference" "C3" (at 108.585 64.77 0)
       (effects (font (size 1.27 1.27)) (justify left))
     )
@@
       (effects (font (size 1.27 1.27)) (justify left))
     )
-    (property "Footprint" "" (at 108.9152 71.12 0)
+    (property "Footprint" "Capacitor_SMD:CP_Elec_5x5.4" (at 108.9152 71.12 0)
       (effects (font (size 1.27 1.27)) hide)
     )
@@
       (project "s13131_breakout"
         (path "/9b830ee6-51b1-4891-8c58-db3625e8ab27"
-          (reference "C?") (unit 1)
+          (reference "C3") (unit 1)
         )
       )

Commit message: Updated breakout board and schematic.
Parts:
- C3: footprint Capacitor_SMD:CP_Elec_5x5.4 -> Capacitor_Tantalum_SMD:CP_EIA-7343-15_Kemet-W_Pad2.25x2.55mm_HandSolder
Changed lines of the file:
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@@
       (effects (font (size 1.27 1.27)) (justify left))
     )
-    (property "Footprint" "Capacitor_SMD:CP_Elec_5x5.4" (at 108.9152 71.12 0)
+    (property "Footprint" "Capacitor_Tantalum_SMD:CP_EIA-7343-15_Kemet-W_Pad2.25x2.55mm_HandSolder" (at 108.9152 71.12 0)
       (effects (font (size 1.27 1.27)) hide)
     )
